File: smart_db_v2/smart_db/smart_db.kicad_sch (KiCad schematic)
At the start: 70 parts, among them J1 AudioJack2, J2 Screw_Terminal_01x02, J3 Conn_01x04_Pin, J4 USB_C_Receptacle_USB2.0_14P, K1 SLA-12VDC-SL-C, Q1 IRLZ44N, Q2 AO3400A, SW1 SW_Push, SW2 SW_Push, SW3 SW_Push, U1 ADS1115IDGS, U2 PC817, U3 AMS1117, U4 ESP32-S3, U5 CP2102N-Axx-xQFN28

Commit message: Implement SmartDB v2 firmware, cloud API and documentation
Parts:
- removed C12, C13, C14: C_US, Capacitor_SMD:C_0805_2012Metric_Pad1.18x1.45mm_HandSolder, symbol Device:C_US
- removed D3, D4: LED, LED_SMD:LED_0805_2012Metric_Pad1.15x1.40mm_HandSolder, symbol Device:LED
- removed F2: Fuse, Fuse:Fuse_0805_2012Metric_Pad1.15x1.40mm_HandSolder, symbol Device:Fuse
- removed FB1: FerriteBead, Ferrite_THT:LairdTech_28C0236-0JW-10, symbol Device:FerriteBead
- removed R10, R11: 330, Resistor_SMD:R_0805_2012Metric_Pad1.20x1.40mm_HandSolder, symbol Device:R_US
- removed R5: 220, Resistor_SMD:R_0805_2012Metric_Pad1.20x1.40mm_HandSolder, symbol Device:R_US
- removed SW1: SW_Push, Button_Switch_SMD:SW_Push_1P1T-MP_NO_Horizontal_Alps_SKRTLAE010, symbol Switch:SW_Push
- removed U2: PC817, Package_DIP:DIP-4_W7.62mm, symbol Isolator:PC817
- added C19: 10uF 10V X7R, Capacitor_SMD:C_0805_2012Metric_Pad1.18x1.45mm_HandSolder, symbol Device:C_US
- added C20: 100nF 10V X7R, Capacitor_SMD:C_0805_2012Metric_Pad1.18x1.45mm_HandSolder, symbol Device:C_US
- added C21: 100nF 25V X7R, Capacitor_SMD:C_0603_1608Metric, symbol Device:C
- added C22, C24: 100uF 10V, Capacitor_SMD:CP_Elec_6.3x7.7, symbol Device:C_Polarized
- added C23: 22uF 10V X7R, Capacitor_SMD:C_1206_3216Metric, symbol Device:C
- added C25: 10uF 16V X7R, Capacitor_SMD:C_0805_2012Metric, symbol Device:C
- added C26: 100nF 16V X7R, Capacitor_SMD:C_0603_1608Metric, symbol Device:C
- added D10, D9: BAT54S, Package_TO_SOT_SMD:SOT-23, symbol Diode:BAT54S
- added H1, H2, H3, H4: M3 mounting, MountingHole:MountingHole_3.2mm_M3, symbol Mechanical:MountingHole
- added J5: TEST_LOAD, TerminalBlock_Phoenix:TerminalBlock_Phoenix_MKDS-1,5-2_1x02_P5.00mm_Horizontal, symbol Connector:Screw_Terminal_01x02
- added J6: CAM USB 5V OUT, SmartDB:USB_A_TE_292303-7_Horizontal_Edge, symbol Connector:USB_A
- added L1: 6.8uH SRP5030TA-6R8M, Inductor_SMD:L_Bourns_SRP5030T, symbol Device:L
- added R26, R27, R28: 100k, Resistor_SMD:R_0805_2012Metric_Pad1.20x1.40mm_HandSolder, symbol Device:R_US
- added R29: 0R 1A min, Resistor_SMD:R_0805_2012Metric, symbol Device:R
- added R30: 10R 1%, Resistor_SMD:R_0603_1608Metric, symbol Device:R
- added TP1: LOGIC_5V_FUSED, TestPoint:TestPoint_Pad_D1.5mm, symbol Connector:TestPoint
- added TP2: VCC, TestPoint:TestPoint_Pad_D1.5mm, symbol Connector:TestPoint
- added TP3: MCU_3V3, TestPoint:TestPoint_Pad_D1.5mm, symbol Connector:TestPoint
- added TP4: ADC_3V3, TestPoint:TestPoint_Pad_D1.5mm, symbol Connector:TestPoint
- added TP5: BGND, TestPoint:TestPoint_Pad_D1.5mm, symbol Connector:TestPoint
- BZ1: value Buzzer -> Buzzer (3V3 type TBD)
- C1: value 100nF -> 220nF
- C10: value C_US -> 100nF
- C11: value C_US -> 1uF
- C15, C18: value 0.1uF -> 100nF; footprint Capacitor_SMD:C_0805_2012Metric_Pad1.18x1.45mm_HandSolder -> Capacitor_SMD:C_0603_1608Metric
- C4: value 1uF -> 10uF 10V X7R; footprint Capacitor_SMD:C_0805_2012Metric_Pad1.18x1.45mm_HandSolder -> Capacitor_SMD:C_0805_2012Metric
- C5: value C_US -> 10uF 10V X7R; footprint Capacitor_SMD:C_0805_2012Metric_Pad1.18x1.45mm_HandSolder -> Capacitor_SMD:C_1206_3216Metric
- C6: value C_US -> 100nF 10V X7R
- C7, C8: value C_US -> 22uF 10V X7R; footprint Capacitor_SMD:C_0805_2012Metric_Pad1.18x1.45mm_HandSolder -> Capacitor_SMD:C_1206_3216Metric
- C9: value C_US -> 10uF
- D1: value 1N4007 -> M7 (1N4007 SMD); footprint Diode_THT:D_DO-41_SOD81_P10.16mm_Horizontal -> Diode_SMD:D_SMA
- D2: value LED -> ADC POWER
- D5: value LED -> POWER
- D6: value LED_KRGB -> SMLVN6RGB1U1; footprint LED_SMD:LED_RGB_5050-6 -> SmartDB:LED_ROHM_SMLVN6_Preview; symbol Device:LED_KRGB -> LED:SMLVN6RGB
- D7: footprint rpi:SOT143 -> Package_TO_SOT_SMD:SOT-143; symbol rpi:SP0503BAHTG -> Power_Protection:SP0503BAHT; AVAILABILITY Good -> (none); Availability In Stock -> (none); Check_prices https://www.snapeda.com/parts/SP0503BAHTG/Littelfuse/view-p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 -> (none); MF Littelfuse Inc. -> (none); MP SP0503BAHTG -> (none); PACKAGE SOT-143 Littelfuse -> (none); PARTREV N/A -> (none); PRICE 0.46 USD -> (none); Package SOT-143 Littelfuse -> (none); Price None -> (none); STANDARD IPC-7351B -> (none); SnapEDA_Link https://www.snapeda.com/parts/SP0503BAHTG/Littelfuse/view-p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 -> (none)
- D8: value LED -> USB BRIDGE POWER
- F1: value Polyfuse -> 046701.5NRHF 1.5A; footprint Fuse:Fuse_0805_2012Metric_Pad1.15x1.40mm_HandSolder -> Fuse:Fuse_0603_1608Metric; symbol Device:Polyfuse -> Device:Fuse
- J1: value AudioJack2 -> SCT-013-000 ONLY; footprint Connector_Audio:Jack_3.5mm_CUI_SJ-3523-SMT_Horizontal -> SmartDB:Jack_3.5mm_SJ-3523-SMT_Local
- J2: value Screw_Terminal_01x02 -> REGULATED 5V INPUT
- J3: value Conn_01x04_Pin -> THERMAL_I2C; footprint Connector_PinHeader_2.54mm:PinHeader_1x04_P2.54mm_Horizontal -> SmartDB:PinHeader_1x04_P2.54mm_Horizontal_Edge
- J4: footprint Connector_USB:USB_C_Receptacle_Amphenol_12401948E412A -> SmartDB:USB_C_Receptacle_Amphenol_12401948E412A_Preview
- K1: value SLA-12VDC-SL-C -> G5LE-1 DC5; footprint rpi:RELAY_SLA-12VDC-SL-C -> Relay_THT:Relay_SPDT_Omron-G5LE-1; symbol rpi:SLA-12VDC-SL-C -> Relay:G5LE-1; Availability Not in stock -> (none); Check_prices https://www.snapeda.com/parts/SLA-12VDC-SL-C/Songle+Relay/v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 -> (none); MANUFACTURER Songle Relay -> (none); MAXIMUM_PACKAGE_HEIGHT 20.4 mm -> (none); MF Songle Relay -> (none); MP SLA-12VDC-SL-C -> (none); Package None -> (none); Price None -> (none); STANDARD Manufacturer Recommendations -> (none); SnapEDA_Link https://www.snapeda.com/parts/SLA-12VDC-SL-C/Songle+Relay/v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 -> (none)
- Q1: value IRLZ44N -> AO3400A; footprint Package_TO_SOT_THT:TO-220-3_Vertical -> Package_TO_SOT_SMD:SOT-23; symbol Transistor_FET:IRLZ44N -> Transistor_FET:AO3400A
- R1, R2: value 10k -> 1k 1%
- R13, R14: value R_US -> 10k
- R15: value R -> 100
- R21: value R_US -> 1k
- R23: value 33 -> 18 ohm 1% 0.25W
- R3, R4: value 10k -> 10k 1%
- SW2: value SW_Push -> BOOT; footprint Button_Switch_SMD:SW_Push_1P1T-MP_NO_Horizontal_Alps_SKRTLAE010 -> Button_Switch_SMD:SW_Push_1P1T_NO_CK_KMR2
- SW3: value SW_Push -> RESET; footprint Button_Switch_SMD:SW_Push_1P1T-MP_NO_Horizontal_Alps_SKRTLAE010 -> Button_Switch_SMD:SW_Push_1P1T_NO_CK_KMR2
- U3: value AMS1117 -> AP63203WU-7; footprint Package_TO_SOT_SMD:SOT-223-3_TabPin2 -> Package_TO_SOT_SMD:TSOT-23-6; symbol Regulator_Linear:AMS1117 -> Regulator_Switching:AP63203WU
- U4: value ESP32-S3 -> ESP32-S3-WROOM-1-N16R8; footprint Package_DFN_QFN:QFN-56-1EP_7x7mm_P0.4mm_EP4x4mm -> SmartDB:ESP32_S3_WROOM_1_Edge; symbol MCU_Espressif:ESP32-S3 -> RF_Module:ESP32-S3-WROOM-1; JLCPCB Part (none) -> C2913202
- U5: value CP2102N-Axx-xQFN28 -> CP2102N-A02-GQFN28
Connections:
- net BGND: now also C10.2, C11.2, C17.2, C18.2, C2.2, C9.2, D5.1 (K), D6.4 (GK), D6.5 (RK), D6.6 (BK), D7.1 (A), J3.3 (Pin_3), Q1.2 (S), Q2.2 (S), R24.2, R25.2, SW2.1, SW3.1, U1.1 (ADDR), U1.6 (AIN2), U1.7 (AIN3), U3.4 (GND), U4.1 (GND), U4.40 (GND), U4.41 (GND), C19.2, C20.2, C22.2, C23.2, C24.2, C25.2, C26.2, D10.1 (A), D9.1 (A), J6.4 (GND), J6.SH (Shield), R26.2, R27.2, R28.2, TP5.1; no longer D7.2, K1.NO, Q1.3 (S), R24.1, R25.1, R3.2, U3.1 (ADJ)
- net CTL: now also R6.1, U4.4 (IO4), R27.1; no longer U4.9 (GPIO4)
- net RX: now also U4.37 (TXD0); no longer U4.49 (U0TXD)
- net SCL: now also U4.38 (IO2); no longer U4.7 (GPIO2)
- net SDA: now also U4.18 (IO10); no longer U4.8 (GPIO3)
- net TX: now also U4.36 (RXD0); no longer U4.50 (U0RXD)
- net VCC: now also C15.1, C16.1, C17.1, C18.1, R22.1, U3.1 (FB), U5.7 (VREGIN), L1.2, R29.1, R30.1, TP2.1; no longer C17.2, C18.2, C3.1, C4.1, R3.1, R4.1, U1.8 (VDD), U3.2 (VO)
- net at U4.11 (IO18): no longer R16.1
- net LED_R_A: now reaches D6.2 (RA), R16.2
- net RELAY_LOW: now reaches D1.2 (A)
- net RELAY_LOW: now also K1.2, Q1.3 (D); no longer K1.C1
- net USB_LED_A: now reaches D8.2 (A), R22.2
- net EN: now reaches SW3.2
- net EN: now also C11.1, R13.2, U4.3 (EN); no longer U4.6 (GPIO1)
- net LOGIC_5V_FUSED: now reaches C5.1, C6.1, F1.2, U3.3 (IN)
- net LOGIC_5V_FUSED: now also D1.1 (K), K1.5, U3.2 (EN), C19.1, C20.1, C22.1, C24.1, C25.1, C26.1, J6.1 (VBUS), TP1.1
- net ADC_LED_A: now reaches D2.2 (A), R9.2
- net USB_VBUS: now reaches D7.4 (K), J4.A4 (VBUS), J4.A9 (VBUS), J4.B4 (VBUS), J4.B9 (VBUS)
- net USB_VBUS: now also R19.1; no longer R19.2, R20.1, U5.8 (VBUS)
- net at U4.10 (IO17): no longer R15.1
- net LED_B: now reaches U4.12 (IO8)
- net LED_B: now also R18.1; no longer R17.2
- net at U4.13 (USB_D-): no longer R18.2
- net MCU_3V3: now reaches BZ1.1 (+), C10.1, C9.1, J3.4 (Pin_4), R12.1, R13.1, R14.1, R7.1, R8.1, U4.2 (3V3)
- net MCU_3V3: now also C23.1, R29.2, TP3.1; no longer C11.1, U4.20 (VDD3P3_RTC), U4.29 (VDD_SPI), U4.3 (VDD3P3), U4.46 (VDD3P3_CPU)
- net BOOT: now reaches U4.27 (IO0)
- net BOOT: now also R14.2, SW2.2
- net BUZZER_DRIVE: now reaches U4.5 (IO5)
- net BUZZER_DRIVE: now also R15.1; no longer SW2.2
- net ADC_AIN1: now reaches R2.2, U1.5 (AIN1)
- net ADC_AIN1: now also C1.2, D10.3 (COM); no longer C2.1
- net RELAY_GATE: now reaches Q1.1 (G), R6.2
- net RELAY_GATE: now also R28.1
- net Net-(D5-A): now reaches D5.2 (A), R12.2
- net USB_RESET: now reaches R21.2, U5.9 (~{RST})
- net LOGIC_5V_IN: now reaches F1.1
- net LOGIC_5V_IN: now also J2.2 (Pin_2)
- net USB_D+: now reaches J4.A6 (D+), J4.B6 (D+), U5.4 (D+)
- net USB_D+: now also D7.2 (K); no longer D7.1
- net USB_D-: now reaches D7.3 (K), J4.A7 (D-), J4.B7 (D-), U5.5 (D-)
- net Net-(Q2-G): now reaches Q2.1 (G), R15.2
- net Net-(Q2-G): now also R26.1
- net LED_G: now reaches R17.1
- net LED_G: now also U4.7 (IO7); no longer D6.3 (GA)
- net BUZZER_LOW: now reaches BZ1.2 (-)
- net BUZZER_LOW: now also Q2.3 (D); no longer Q2.2 (S)
- net USB_CC2: now reaches J4.B5 (CC2)
- net USB_CC2: now also R25.1; no longer R24.2
- net USB_CC1: now reaches J4.A5 (CC1)
- net USB_CC1: now also R24.1; no longer R25.2
- removed net BVCC: J2.2 (Pin_2), K1.NC
- removed net IO0: D5.1 (K), D6.1 (K), Q2.3 (D), R13.2, R14.2, SW2.1, SW3.1, U4.4 (CHIP_PU), U4.57 (GND)
- removed net PGND: C1.2, C2.2, J1.T, R23.2, U1.1 (ADDR), U1.2 (ALERT/RDY), U1.6 (AIN2), U1.7 (AIN3)
- removed net PVCC: C1.1, J1.S, K1.COM1, K1.COM2, R1.2, R23.1
- new net ADC_3V3: C3.1, C4.1, D10.2 (K), D9.2 (K), R3.1, R30.2, TP4.1, U1.8 (VDD)
- new net ADC_AIN0: C1.1, D9.3 (COM), R1.2, U1.4 (AIN0)
- new net BUCK_BST: C21.1, U3.6 (BST)
- new net BUCK_SW: C21.2, L1.1, U3.5 (SW)
- new net CT_BIAS: C2.1, J1.S, R2.1, R23.2, R3.2, R4.1
- new net CT_HI: J1.T, R1.1, R23.1
- new net LED_B_A: D6.1 (BA), R18.2
- new net LED_G_A: D6.3 (GA), R17.2
- new net LED_R: R16.1, U4.6 (IO6)
- new net LOAD_IN: J5.1 (Pin_1), K1.1
- new net LOAD_OUT: J5.2 (Pin_2), K1.3
- new net USB_VBUS_SENSE: R19.2, R20.1, U5.8 (VBUS)
- no-connect marks 0 -> 49
Other:
- note added: "01 POWER / 5 V TO 3.3 V"
- note added: "02 USB / UART PROGRAMMING"
- note added: "03 ESP32-S3 / BOOT / RESET"
- note added: "04 CT / ADC ANALOG FRONT END"
- note added: "05 RELAY / TEST LOAD"
- note added: "06 INDICATORS / EXTERNAL I2C"
- note added: "3.3 V logic only. Buzzer part selection and bench measurements pending."
- note added: "AC current transformer only. Differential AIN0-AIN1, address 0x48."
- note added: "ESP32-S3-WROOM-1-N16R8. Module RF keepout on every copper layer."
- note added: "J2 regulated 5 V only. Buck + local reservoirs. Not battery charging."
- note added: "J6 USB-A: camera 5V POWER OUT. D-/D+ NC; GND and shell to BGND. USB-A to micro-USB cable powers external ESP32-CAM-MB base. Wi-Fi image transfer requires firmware. Shared F1 1.5A fuse; camera/base budget 0.5A, total target <=1.1A at 25C; verify at temperature."
- note added: "MECHANICAL + MEASUREMENT POINTS"
- note added: "Normally-open dry contact loop. 5-24 V DC / 1 A resistive bench target."
- note added: "USB is data only; J2 powers the board. Hold BOOT, pulse RESET."
- title: (none) -> SmartDB v2 - low-voltage bench revision
- moved on the sheet: BZ1, C1, C10, C11, C15, C16, C17, C18, C2, C3, C4, C5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
